File: Adafruit RGB Matrix HAT.sch (EAGLE design)
At the start: 38 parts, among them IC3 MAX4866T, Q1 AOD514, Q2 AOD417, U1 CAT24C32, U2 2.1MMJACKSMT, U3 74AHCT245, U4 DS1307, U5 74AHCT245, Y1 32.768kHz

Commit message: Update to Rev C
Parts:
- removed U2: 2.1MMJACKSMT, adafruit:2.1MMJACKSMT
- added JP1: (no value), pinhead-ez:PINHD-1X1
- added SJ2: (no value), microbuilder:SOLDERJUMPER_2WAY
- added X1: 2.1mm DC, adafruit_electromech:DCBARRELSMT
- added Y2: 32.768kHz, microbuilder:CRYSTAL_3215
- FID1, FID2, FID3: value FIDUCIAL"" -> FIDUCIAL_1MM; device microbuilder:FIDUCIAL"" -> microbuilder:FIDUCIAL_1MM
- Q2: device transistor-power:IRFR5305 -> microbuilder:MOSFET-PTO252
- RPI1: device microbuilder:RASPBERRYPI_BPLUS_HATSLOTS -> adafruit_sbc:RASPBERRYPI_BPLUS_HATSLOTS
- U1: device microbuilder:EEPROM_I2C_SOIC8_GENERIC -> microbuilder:EEPROM_I2C_8PIN_GENERIC
- U3, U5: device microbuilder:74LCX245 -> microbuilder:74LCX245_TSSOP20
Connections:
- new net M1_E: SJ2.2, U3.B3
- new net M1_E': JP15.8, SJ2.1
- new net M1_E'': JP15.16, SJ2.3
- net 5VIN: now also X1.PWR; no longer U2.TIP
- net GND: now also X1.GND, X1.GNDBREAK; no longer JP15.16, JP15.8, U2.RING, U2.RING_SW, U3.A3
- net GPIO24: now also JP1.1, U3.A3
- net N$2: now also Y2.1
- net N$3: now also Y2.2
